Commit message: Planning succeeds; fix base planning randomization seed.

File: predicators/envs/assets/urdf/igibson_fetch_description/robots/fetch.urdf (robot description, URDF)
Before this commit: robot fetch, 27 links, 26 joints
Links:
- link r_gripper_finger_link: geometry collision box size=0.055 0.013 0.026; visual box size=0.055 0.013 0.026
